File: mini/keyboard-mini/keyboard-mini.kicad_sch (KiCad schematic)
At the start: 37 parts, among them J2 IO

Commit message: mini
Parts:
- D_1, D_2, D_3, D_4, D_5, D_6, D_7, D_8, D_9: footprint Diode_THT:D_DO-35_SOD27_P7.62mm_Horizontal -> EUK:D_DO-35_SOD27_P7.62mm_Horizontal
Changed lines of the file:
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@@
 			)
 		)
-		(property "Footprint" "Diode_THT:D_DO-35_SOD27_P7.62mm_Horizontal"
+		(property "Footprint" "EUK:D_DO-35_SOD27_P7.62mm_Horizontal"
 			(at 50.8 60.96 0)
 			(effects
@@
 			)
 		)
-		(property "Footprint" "Diode_THT:D_DO-35_SOD27_P7.62mm_Horizontal"
+		(property "Footprint" "EUK:D_DO-35_SOD27_P7.62mm_Horizontal"
 			(at 76.2 60.96 0)
 			(effects
@@
 			)
 		)
-		(property "Footprint" "Diode_THT:D_DO-35_SOD27_P7.62mm_Horizontal"
+		(property "Footprint" "EUK:D_DO-35_SOD27_P7.62mm_Horizontal"
 			(at 50.8 86.36 0)
 			(effects
@@
 			)
 		)
-		(property "Footprint" "Diode_THT:D_DO-35_SOD27_P7.62mm_Horizontal"
+		(property "Footprint" "EUK:D_DO-35_SOD27_P7.62mm_Horizontal"
 			(at 76.2 86.36 0)
 			(effects
@@
 			)
 		)
-		(property "Footprint" "Diode_THT:D_DO-35_SOD27_P7.62mm_Horizontal"
+		(property "Footprint" "EUK:D_DO-35_SOD27_P7.62mm_Horizontal"
 			(at 76.2 106.68 0)
 			(effects
@@
 			)
 		)
-		(property "Footprint" "Diode_THT:D_DO-35_SOD27_P7.62mm_Horizontal"
+		(property "Footprint" "EUK:D_DO-35_SOD27_P7.62mm_Horizontal"
 			(at 50.8 106.68 0)
 			(effects
@@
 			)
 		)
-		(property "Footprint" "Diode_THT:D_DO-35_SOD27_P7.62mm_Horizontal"
+		(property "Footprint" "EUK:D_DO-35_SOD27_P7.62mm_Horizontal"
 			(at 104.14 86.36 0)
 			(effects
@@
 			)
 		)
-		(property "Footprint" "Diode_THT:D_DO-35_SOD27_P7.62mm_Horizontal"
+		(property "Footprint" "EUK:D_DO-35_SOD27_P7.62mm_Horizontal"
 			(at 104.14 106.68 0)
 			(effects
@@
 			)
 		)
-		(property "Footprint" "Diode_THT:D_DO-35_SOD27_P7.62mm_Horizontal"
+		(property "Footprint" "EUK:D_DO-35_SOD27_P7.62mm_Horizontal"
 			(at 104.14 60.96 0)
 			(effects
