File: split/pcb/keyboard.kicad_pcb (KiCad board)
At the start: 2 copper layers, 163.5 x 129.2 mm, 115 parts, among them J1 TRRS, J2 IO, J3 IO

Commit message: pcb tweaks
Other:
- board text added: "I2C1_SCL"
- board text added: "I2C1_SDA"
Changed lines of the file:
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@@
+		)
+	)
+	(gr_text "I2C1_SCL"
+		(at 321.5 201 90)
+		(layer "F.SilkS")
+		(effects
+			(font
+				(size 1 1)
+				(thickness 0.15)
+			)
+			(justify left bottom)
 		)
 	)
@@
 		)
 	)
+	(gr_text "I2C1_SDA"
+		(at 316.5 201 90)
+		(layer "F.SilkS")
+		(effects
+			(font
+				(size 1 1)
+				(thickness 0.15)
+			)
+			(justify left bottom)
+		)
+	)
 	(gr_text "IO1"
 		(at 313.75 189.25 90)
@@
 		)
 	)
+	(gr_text "I2C1_SCL"
+		(at 316.5 190 90)
+		(layer "B.SilkS")
+		(effects
+			(font
+				(size 1 1)
+				(thickness 0.15)
+			)
+			(justify left bottom mirror)
+		)
+	)
 	(gr_text "GP22"
 		(at 316.5 197 90)
@@
 		)
 	)
+	(gr_text "I2C1_SDA"
+		(at 321.5 190 90)
+		(layer "B.SilkS")
+		(effects
+			(font
+				(size 1 1)
+				(thickness 0.15)
+			)
+			(justify left bottom mirror)
+		)
+	)
 	(gr_text "3V3"
 		(at 306.25 201 90)
@@
 	)
 	(segment
+		(start 185.325 221.31125)
+		(end 187.51375 223.5)
+		(width 0.25)
+		(layer "B.Cu")
+		(net 3)
+	)
+	(segment
+		(start 187.36375 185.25)
+		(end 196.25 185.25)
+		(width 0.25)
+		(layer "B.Cu")
+		(net 3)
+	)
+	(segment
+		(start 187.46375 242.5)
+		(end 196.25 242.5)
+		(width 0.25)
+		(layer "B.Cu")
+		(net 3)
+	)
+	(segment
+		(start 225.626427 141.848)
+		(end 218.724427 148.75)
+		(width 0.25)
+		(layer "B.Cu")
+		(net 3)
+	)
+	(segment
+		(start 187.41375 166.25)
+		(end 197 166.25)
+		(width 0.25)
+		(layer "B.Cu")
+		(net 3)
+	)
+	(segment
 		(start 281.375 144.5)
 		(end 278.723 141.848)
@@
 	)
 	(segment
-		(start 185.325 221.31125)
-		(end 187.51375 223.5)
-		(width 0.25)
-		(layer "B.Cu")
-		(net 3)
-	)
-	(segment
-		(start 225.626427 141.848)
-		(end 218.724427 148.75)
-		(width 0.25)
-		(layer "B.Cu")
-		(net 3)
-	)
-	(segment
-		(start 187.36375 185.25)
-		(end 196.25 185.25)
+		(start 278.723 141.848)
+		(end 225.626427 141.848)
+		(width 0.25)
+		(layer "B.Cu")
+		(net 3)
+	)
+	(segment
+		(start 185.325 164.16125)
+		(end 185.325 240.36125)
+		(width 0.25)
+		(layer "B.Cu")
+		(net 3)
+	)
+	(segment
+		(start 304.25 144.5)
+		(end 281.375 144.5)
+		(width 0.25)
+		(layer "B.Cu")
+		(net 3)
+	)
+	(segment
+		(start 310.08 150.33)
+		(end 304.25 144.5)
+		(width 0.25)
+		(layer "B.Cu")
+		(net 3)
+	)
+	(segment
+		(start 185.325 240.36125)
+		(end 187.46375 242.5)
+		(width 0.25)
+		(layer "B.Cu")
+		(net 3)
+	)
+	(segment
+		(start 185.325 202.26125)
+		(end 187.56375 204.5)
+		(width 0.25)
+		(layer "B.Cu")
+		(net 3)
+	)
+	(segment
+		(start 185.325 153.675)
+		(end 185.325 164.16125)
+		(width 0.25)
+		(layer "B.Cu")
+		(net 3)
+	)
+	(segment
+		(start 187.51375 223.5)
+		(end 196.25 223.5)
+		(width 0.25)
+		(layer "B.Cu")
+		(net 3)
+	)
+	(segment
+		(start 185.325 183.21125)
+		(end 187.36375 185.25)
+		(width 0.25)
+		(layer "B.Cu")
+		(net 3)
+	)
+	(segment
+		(start 218.724427 148.75)
+		(end 190.25 148.75)
 		(width 0.25)
 		(layer "B.Cu")
@@
 	)
 	(segment
-		(start 185.325 153.675)
-		(end 185.325 164.16125)
-		(width 0.25)
-		(layer "B.Cu")
-		(net 3)
-	)
-	(segment
-		(start 187.46375 242.5)
-		(end 196.25 242.5)
-		(width 0.25)
-		(layer "B.Cu")
-		(net 3)
-	)
-	(segment
-		(start 218.724427 148.75)
-		(end 190.25 148.75)
-		(width 0.25)
-		(layer "B.Cu")
-		(net 3)
-	)
-	(segment
-		(start 187.41375 166.25)
-		(end 197 166.25)
-		(width 0.25)
-		(layer "B.Cu")
-		(net 3)
-	)
-	(segment
 		(start 185.325 164.16125)
-		(end 185.325 240.36125)
-		(width 0.25)
-		(layer "B.Cu")
-		(net 3)
-	)
-	(segment
-		(start 304.25 144.5)
-		(end 281.375 144.5)
-		(width 0.25)
-		(layer "B.Cu")
-		(net 3)
-	)
-	(segment
-		(start 310.08 150.33)
-		(end 304.25 144.5)
-		(width 0.25)
-		(layer "B.Cu")
-		(net 3)
-	)
-	(segment
-		(start 185.325 240.36125)
-		(end 187.46375 242.5)
-		(width 0.25)
-		(layer "B.Cu")
-		(net 3)
-	)
-	(segment
-		(start 185.325 202.26125)
-		(end 187.56375 204.5)
+		(end 187.41375 166.25)
 		(width 0.25)
 		(layer "B.Cu")
@@
 		(width 0.25)
 		(layer "B.Cu")
-		(net 3)
-	)
-	(segment
-		(start 187.51375 223.5)
-		(end 196.25 223.5)
-		(width 0.25)
-		(layer "B.Cu")
-		(net 3)
-	)
-	(segment
-		(start 185.325 183.21125)
-		(end 187.36375 185.25)
-		(width 0.25)
-		(layer "B.Cu")
-		(net 3)
-	)
-	(segment
-		(start 185.325 164.16125)
-		(end 187.41375 166.25)
-		(width 0.25)
-		(layer "B.Cu")
-		(net 3)
-	)
-	(segment
-		(start 278.723 141.848)
-		(end 225.626427 141.848)
-		(width 0.25)
-		(layer "B.Cu")

Commit message: missing changes
Parts:
- moved H6 1.25 mm to (182.5, 148.8)
- moved H4 1.12 mm to (182.5, 245.5)
Routing:
- net GND: vias 273 -> 272
Other:
- board size 163.5 x 129.2 mm -> 161.8 x 129.2 mm
- board text added: "The Extremely Unnecessary Keyboard -> Rev .2"
- board text removed: "The Extremely Unnecessary Keyboard"
